File: oswRAKwisBlock.kicad_sch (KiCad schematic)
At the start: 39 parts, among them J1 WisBlock, J2 0524352471, J4 10114830-10102LF, J5 USB micro, Q1 SI1308EDL-T1-GE3, U1 MCP73811T-420I/OT, U5 MIC5365-3.0YC5-TR

Commit message: Finishing up the layout.
Parts:
- C1, C10, C11, C12, C13, C2, C3, C4, C5, C6, C7: footprint AllardChip:CAPC100X50X60L25L -> AllardChip:CAPC100X50X60L25N
- C16: footprint AllardChip:CAPC60X30X39L17L -> AllardChip:CAPC60X30X39L17N
- C8, C9: footprint AllardChip:CAPC200X125X145L45L -> AllardChip:CAPC200X125X145L45N
- L2: footprint AllardChip:INDC400X400X120L120L -> AllardChip:INDC400X400X120L120N
- R1, R2, R3, R4, R5, R8: footprint AllardChip:RESC40X20X15L10L -> AllardChip:RESC40X20X15L10N
- U5: footprint AllardSOT:SOT23-5P65_210X110L33X22L -> AllardSOT:SOT23-5P65_210X110L33X22N
Connections:
- net BTN1: now also J1.32 (IO4); no longer J1.30 (IO2)
- net BTN2: now also J1.30 (IO2); no longer J1.32 (IO4)
- net VDD: now also J1.17 (VDD), J1.18 (VDD)
Other:
- moved on the sheet: C1, C13, C2, C3, C4, C5, C7, U5

Commit message: a couple minor tweaks to the layout (better trace connections) and moving a hole to be in the proper location
Parts:
- added R9: 0, AllardChip:RESC60X30X26L15N, symbol AllardPassive:R00001-10000
Connections:
- net VUSB_BUS: now also R9.1; no longer J1.9 (VBUS)
- new net: J1.9 (VBUS), R9.2
Changed lines of the file:
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@@
 	(wire
 		(pts
-			(xy 54.61 85.09) (xy 54.61 69.85)
+			(xy 54.61 85.09) (xy 54.61 71.12)
 		)
 		(stroke
@@
 	(wire
 		(pts
+			(xy 54.61 66.04) (xy 54.61 62.23)
+		)
+		(stroke
+			(width 0)
+			(type default)
+		)
+	)
+	(wire
+		(pts
 			(xy 198.12 133.35) (xy 198.12 137.16)
 		)
@@
 	)
 	(symbol
+		(lib_id "AllardPassive:R00001-10000")
+		(at 54.61 68.58 0)
+		(unit 1)
+		(exclude_from_sim no)
+		(in_bom yes)
+		(on_board yes)
+		(dnp no)
+		(fields_autoplaced yes)
+		(property "Reference" "R9"
+			(at 55.88 67.3099 0)
+			(effects
+				(font
+					(size 1.27 1.27)
+				)
+				(justify left)
+			)
+		)
+		(property "Value" "0"
+			(at 55.88 69.8499 0)
+			(effects
+				(font
+					(size 1.27 1.27)
+				)
+				(justify left)
+			)
+		)
+		(property "Footprint" "AllardChip:RESC60X30X26L15N"
+			(at 55.626 68.834 90)
+			(effects
+				(font
+					(size 1.27 1.27)
+				)
+				(hide yes)
+			)
+		)
+		(property "Datasheet" "https://industrial.panasonic.com/cdbs/www-data/pdf/RDA0000/AOA0000C301.pdf"
+			(at 54.61 68.58 0)
+			(effects
+				(font
+					(size 1.27 1.27)
+				)
+				(hide yes)
+			)
+		)
+		(property "Description" "0 0201 0.05W 1% Res"
+			(at 54.61 68.58 0)
+			(effects
+				(font
+					(size 1.27 1.27)
+				)
+				(hide yes)
+			)
+		)
+		(property "AI_PN" "${SYMBOL_NAME}"
+			(at 54.61 68.58 0)
+			(effects
+				(font
+					(size 1.2446 1.2446)
+				)
+				(hide yes)
+			)
+		)
+		(property "MPN" "ERJ-1GN0R00C"
+			(at 54.61 68.58 0)
+			(effects
+				(font
+					(size 1.2446 1.2446)
+				)
+				(hide yes)
+			)
+		)
+		(property "Manufacturer" "Panasonic Electronics Components"
+			(at 54.61 68.58 0)
+			(effects
+				(font
+					(size 1.2446 1.2446)
+				)
+				(hide yes)
+			)
+		)
+		(property "manf#" "ERJ-1GN0R00C"
+			(at 54.61 68.58 0)
+			(effects
+				(font
+					(size 1.2446 1.2446)
+				)
+				(hide yes)
+			)
+		)
+		(property "SUP1" "Digi-Key"
+			(at 54.61 68.58 0)
+			(effects
+				(font
+					(size 1.2446 1.2446)
+				)
+				(hide yes)
+			)
+		)
+		(property "SUP1_PN" "P15979CT-ND"
+			(at 54.61 68.58 0)
+			(effects
+				(font
+					(size 1.2446 1.2446)
+				)
+				(hide yes)
+			)
+		)
+		(property "SUP2" "Mouser"
+			(at 54.61 68.58 0)
+			(effects
+				(font
+					(size 1.2446 1.2446)
+				)
+				(hide yes)
+			)
+		)
+		(property "SUP2_PN" "667-ERJ-1GN0R00C"
+			(at 54.61 68.58 0)
+			(effects
+				(font
+					(size 1.2446 1.2446)
+				)
+				(hide yes)
+			)
+		)
+		(property "Tolerance" "1%"
+			(at 54.61 68.58 0)
+			(effects
+				(font
+					(size 1.2446 1.2446)
+				)
+				(hide yes)
+			)
+		)
+		(property "Power" "0.05W"
+			(at 54.61 68.58 0)
+			(effects
+				(font
+					(size 1.2446 1.2446)
+				)
+				(hide yes)
+			)
+		)
+		(property "Temperature" "-55-125"
+			(at 54.61 68.58 0)
+			(effects
+				(font
+					(size 1.2446 1.2446)
+				)
+				(hide yes)
+			)
+		)
+		(property "variant" "default"
+			(at 54.61 68.58 0)
+			(effects
+				(font
+					(size 1.27 1.27)
+				)
+				(hide yes)
+			)
+		)
+		(property "TempCoef" "±200ppm/°C"
+			(at 54.61 68.58 0)
+			(effects
+				(font
+					(size 1.27 1.27)
+				)
+				(hide yes)
+			)
+		)
+		(property "SUP3" "LCSC"
+			(at 54.61 68.58 0)
+			(effects
+				(font
+					(size 1.27 1.27)
+				)
+				(hide yes)
+			)
+		)
+		(property "SUP3_PN" "C716999"
+			(at 54.61 68.58 0)
+			(effects
+				(font
+					(size 1.27 1.27)
+				)
+				(hide yes)
+			)
+		)
+		(pin "1"
+		)
+		(pin "2"
+		)
+		(instances
+			(project "oswRAKwisBlock"
+				(path "/2fe076e6-bb0e-436f-836d-ec5f0ee79cef"
+					(reference "R9")
+					(unit 1)
+				)
+			)
+		)
+	)
+	(symbol
 		(lib_name "R10020-10000_2")
 		(lib_id "AllardPassive:R10020-10000")
@@
 	(symbol
 		(lib_id "power:VDD")
-		(at 54.61 69.85 0)
+		(at 54.61 62.23 0)
 		(unit 1)
 		(exclude_from_sim no)
@@
 		(fields_autoplaced yes)
 		(property "Reference" "#PWR019"
-			(at 54.61 73.66 0)
+			(at 54.61 66.04 0)
 			(effects
 				(font
@@
 		)
 		(property "Value" "VUSB_BUS"
-			(at 54.61 64.77 0)
+			(at 54.61 57.15 0)
 			(effects
 				(font
@@
 		)
 		(property "Footprint" ""
-			(at 54.61 69.85 0)
+			(at 54.61 62.23 0)
 			(effects
 				(font
@@
 		)
 		(property "Datasheet" ""
-			(at 54.61 69.85 0)
+			(at 54.61 62.23 0)
 			(effects
 				(font
@@
 		)
 		(property "Description" "Power symbol creates a global label with name \"VDD\""
-			(at 54.61 69.85 0)
+			(at 54.61 62.23 0)
 			(effects
 				(font
